File: 51.kicad_pcb (KiCad board)
At the start: 2 copper layers, 43 parts, among them J1 Conn_01x04, J2 Conn_01x04, J3 Conn_02x07_Odd_Even, J4 Conn_02x08_Odd_Even, J5 Conn_02x08_Odd_Even, J6 Conn_02x08_Odd_Even, J7 Conn_02x08_Odd_Even, J8 Conn_01x04, J9 Conn_01x04, SW1 SW_Push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

Commit message: V0.1 COMPLETE
Routing:
- net GND: track 14.1 -> 354.1 mm, vias 0 -> 107
- net +5V: track 55.6 -> 169.1 mm, vias 0 -> 4
- net /RST: track 4.43 -> 64.8 mm, vias 0 -> 2
- net /P3.0: track 46.9 -> 102.2 mm
- net /P4.4: track 0.00 -> 31.9 mm, vias 0 -> 1
- net /P4.0: track 0.00 -> 31.4 mm, vias 0 -> 1
- net /P4.5: track 0.00 -> 29.6 mm, vias 0 -> 1
- net /P4.3: track 0.00 -> 29.3 mm, vias 0 -> 1
- net /KEY1: track 44.9 -> 73.4 mm, vias 0 -> 1
- net /P3.1: track 55.9 -> 84.2 mm
- net /P4.1: track 0.00 -> 27.2 mm, vias 0 -> 1
- net /P4.6: track 5.02 -> 29.7 mm, vias 0 -> 1
- net Net-(D1-Pad1): track 0.00 -> 16.2 mm, vias 0 -> 2
- net Net-(C2-Pad2): track 0.00 -> 12.0 mm
- net VBUS: track 15.6 -> 23.6 mm
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- added copper zone on B.Cu, net GND
- added copper zone on F.Cu, net GND
Other:
- board outline added: 80 x 55 mm
- board text added: "JLCJLCJLCJLC"
- board text added: "TYF_V0.1"

Commit message: V0.1.1 加引脚丝印
Routing:
- net (no net): vias 0 -> 5
Other:
- board text added: "5V"
- board text added: "GND"
- board text added: "P0.0"
- board text added: "P0.1"
- board text added: "P0.2"
- board text added: "P0.3"
- board text added: "P0.4"
- board text added: "P0.5"
- board text added: "P0.6"
- board text added: "P0.7"
- board text added: "P1.0"
- board text added: "P1.1"
- board text added: "P1.2"
- board text added: "P1.3"
- board text added: "P1.4"
- board text added: "P1.5"
- board text added: "P1.6"
- board text added: "P1.7"
- board text added: "P2.0"
- board text added: "P2.1"
- board text added: "P2.2"
- board text added: "P2.3"
- board text added: "P2.4"
- board text added: "P2.5"
- board text added: "P2.6"
- board text added: "P2.7"
- board text added: "P3.0"
- board text added: "P3.1"
- board text added: "P3.2"
- board text added: "P3.3"
- board text added: "P3.4"
- board text added: "P3.5"
- board text added: "P3.6"
- board text added: "P3.7"
- board text added: "P4.0"
- board text added: "P4.1"
- board text added: "P4.2"
- board text added: "P4.3"
- board text added: "P4.4"
- board text added: "P4.5"
- board text added: "P4.6"
Changed lines of the file:
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@@
     (effects (font (size 1 1) (thickness 0.15)) (justify mirror))
   )
+  (gr_text "P3.4\n" (at 134.8 111.7 270) (layer "F.SilkS")
+    (effects (font (size 1 1) (thickness 0.15)))
+  )
+  (gr_text "P1.5" (at 115.8 111.6 270) (layer "F.SilkS")
+    (effects (font (size 1 1) (thickness 0.15)))
+  )
+  (gr_text "P0.4" (at 112.1 73.1 270) (layer "F.SilkS")
+    (effects (font (size 1 1) (thickness 0.15)))
+  )
+  (gr_text "P2.2\n" (at 136.3 73.2 270) (layer "F.SilkS")
+    (effects (font (size 1 1) (thickness 0.15)))
+  )
+  (gr_text "P0.7" (at 119.7 73.2 270) (layer "F.SilkS")
+    (effects (font (size 1 1) (thickness 0.15)))
+  )
+  (gr_text "P4.2" (at 98.7 107.2) (layer "F.SilkS")
+    (effects (font (size 1 1) (thickness 0.15)))
+  )
+  (gr_text "GND" (at 103.3 81.2) (layer "F.SilkS")
+    (effects (font (size 1 1) (thickness 0.15)))
+  )
+  (gr_text "P0.5" (at 114.8 73.2 270) (layer "F.SilkS")
+    (effects (font (size 1 1) (thickness 0.15)))
+  )
+  (gr_text "P2.7" (at 123.6 73.2 270) (layer "F.SilkS")
+    (effects (font (size 1 1) (thickness 0.15)))
+  )
+  (gr_text "P2.0" (at 141.3 73.2 270) (layer "F.SilkS")
+    (effects (font (size 1 1) (thickness 0.15)))
+  )
+  (gr_text "P4.3" (at 98.7 109.7) (layer "F.SilkS")
+    (effects (font (size 1 1) (thickness 0.15)))
+  )
+  (gr_text "P1.6\n" (at 118.5 111.7 270) (layer "F.SilkS")
+    (effects (font (size 1 1) (thickness 0.15)))
+  )
+  (gr_text "P0.0" (at 101.9 73.1 270) (layer "F.SilkS")
+    (effects (font (size 1 1) (thickness 0.15)))
+  )
+  (gr_text "P3.7" (at 142.6 111.7 270) (layer "F.SilkS")
+    (effects (font (size 1 1) (thickness 0.15)))
+  )
+  (gr_text "P0.1" (at 104.5 73.1 270) (layer "F.SilkS")
+    (effects (font (size 1 1) (thickness 0.15)))
+  )
+  (gr_text "GND" (at 103.3 86.4) (layer "F.SilkS")
+    (effects (font (size 1 1) (thickness 0.15)))
+  )
+  (gr_text "P4.4" (at 98.7 102.2) (layer "F.SilkS")
+    (effects (font (size 1 1) (thickness 0.15)))
+  )
+  (gr_text "P0.2" (at 107 73.1 270) (layer "F.SilkS")
+    (effects (font (size 1 1) (thickness 0.15)))
+  )
+  (gr_text "P3.5\n" (at 137.4 111.7 270) (layer "F.SilkS")
+    (effects (font (size 1 1) (thickness 0.15)))
+  )
+  (gr_text "P1.0\n" (at 103.2 111.6 270) (layer "F.SilkS")
+    (effects (font (size 1 1) (thickness 0.15)))
+  )
+  (gr_text "P2.1" (at 138.6 73.2 270) (layer "F.SilkS")
+    (effects (font (size 1 1) (thickness 0.15)))
+  )
+  (gr_text "P2.6" (at 126.1 73.2 270) (layer "F.SilkS")
+    (effects (font (size 1 1) (thickness 0.15)))
+  )
+  (gr_text "5V" (at 102.9 89) (layer "F.SilkS")
+    (effects (font (size 1 1) (thickness 0.15)))
+  )
+  (gr_text "P3.3" (at 132.3 111.6 270) (layer "F.SilkS")
+    (effects (font (size 1 1) (thickness 0.15)))
+  )
+  (gr_text "P1.7" (at 120.9 111.7 270) (layer "F.SilkS")
+    (effects (font (size 1 1) (thickness 0.15)))
+  )
+  (gr_text "P0.6" (at 117.2 73.2 270) (layer "F.SilkS")
+    (effects (font (size 1 1) (thickness 0.15)))
+  )
+  (gr_text "P2.3" (at 133.6 73.2 270) (layer "F.SilkS")
+    (effects (font (size 1 1) (thickness 0.15)))
+  )
+  (gr_text "5V" (at 102.8 83.7) (layer "F.SilkS")
+    (effects (font (size 1 1) (thickness 0.15)))
+  )
+  (gr_text "P3.0\n" (at 124.8 111.6 270) (layer "F.SilkS")
+    (effects (font (size 1 1) (thickness 0.15)))
+  )
+  (gr_text "P1.1" (at 105.7 111.6 270) (layer "F.SilkS")
+    (effects (font (size 1 1) (thickness 0.15)))
+  )
+  (gr_text "P4.5" (at 98.7 99.6) (layer "F.SilkS")
+    (effects (font (size 1 1) (thickness 0.15)))
+  )
+  (gr_text "P3.1" (at 127.8 111.6 270) (layer "F.SilkS")
+    (effects (font (size 1 1) (thickness 0.15)))
+  )
+  (gr_text "P3.2" (at 130 111.6 270) (layer "F.SilkS")
+    (effects (font (size 1 1) (thickness 0.15)))
+  )
+  (gr_text "P1.3" (at 110.8 111.6 270) (layer "F.SilkS")
+    (effects (font (size 1 1) (thickness 0.15)))
+  )
+  (gr_text "P4.1" (at 98.7 96.9) (layer "F.SilkS")
+    (effects (font (size 1 1) (thickness 0.15)))
+  )
+  (gr_text "P1.4" (at 113.3 111.6 270) (layer "F.SilkS")
+    (effects (font (size 1 1) (thickness 0.15)))
+  )
+  (gr_text "P2.4" (at 131.1 73.2 270) (layer "F.SilkS")
+    (effects (font (size 1 1) (thickness 0.15)))
+  )
+  (gr_text "P2.5" (at 128.5 73.2 270) (layer "F.SilkS")
+    (effects (font (size 1 1) (thickness 0.15)))
+  )
+  (gr_text "P1.2\n" (at 108.3 111.6 270) (layer "F.SilkS")
+    (effects (font (size 1 1) (thickness 0.15)))
+  )
+  (gr_text "P0.3" (at 109.6 73.1 270) (layer "F.SilkS")
+    (effects (font (size 1 1) (thickness 0.15)))
+  )
+  (gr_text "P4.6" (at 98.7 94.5) (layer "F.SilkS")
+    (effects (font (size 1 1) (thickness 0.15)))
+  )
+  (gr_text "P4.0" (at 98.7 104.7) (layer "F.SilkS")
+    (effects (font (size 1 1) (thickness 0.15)))
+  )
+  (gr_text "P3.6" (at 140 111.7 270) (layer "F.SilkS")
+    (effects (font (size 1 1) (thickness 0.15)))
+  )
+  (via (at 110.4 75.7) (size 0.8) (drill 0.4) (layers "F.Cu" "B.Cu") (free) (net 0))
+  (via (at 162.7 75.6) (size 0.8) (drill 0.4) (layers "F.Cu" "B.Cu") (free) (net 0))
+  (via (at 94.1 91.8) (size 0.8) (drill 0.4) (layers "F.Cu" "B.Cu") (free) (net 0))
+  (via (at 110.5 82.1) (size 0.8) (drill 0.4) (layers "F.Cu" "B.Cu") (free) (net 0))
+  (via (at 160.4 76.1) (size 0.8) (drill 0.4) (layers "F.Cu" "B.Cu") (free) (net 0))
   (segment (start 167 84.7) (end 167 86.95) (width 0.508) (layer "F.Cu") (net 1))
   (segment (start 157.1 96.15) (end 158.65 96.15) (width 0.508) (layer "F.Cu") (net 1))
